File: first schematic.kicad_sch (KiCad schematic)
At the start: 9 parts, among them SW1 SW_DPDT_x2, U1 ATtiny85V-10P

Commit message: Autosave
Parts:
- removed unit 2 of SW1
Other:
- moved on the sheet: SW1A
Changed lines of the file:
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@@
-	)
-	(symbol
-		(lib_id "Switch:SW_DPDT_x2")
-		(at 190.5 105.41 0)
-		(unit 2)
-		(body_style 1)
-		(exclude_from_sim no)
-		(in_bom yes)
-		(on_board yes)
-		(in_pos_files yes)
-		(dnp no)
-		(fields_autoplaced yes)
-		(property "Reference" "SW1"
-			(at 190.5 96.52 0)
-			(show_name no)
-			(do_not_autoplace no)
-			(effects
-				(font
-					(size 1.27 1.27)
-				)
-			)
-		)
-		(property "Value" "SW_DPDT_x2"
-			(at 190.5 99.06 0)
-			(show_name no)
-			(do_not_autoplace no)
-			(effects
-				(font
-					(size 1.27 1.27)
-				)
-			)
-		)
-		(property "Footprint" ""
-			(at 190.5 105.41 0)
-			(hide yes)
-			(show_name no)
-			(do_not_autoplace no)
-			(effects
-				(font
-					(size 1.27 1.27)
-				)
-			)
-		)
-		(property "Datasheet" ""
-			(at 190.5 105.41 0)
-			(hide yes)
-			(show_name no)
-			(do_not_autoplace no)
-			(effects
-				(font
-					(size 1.27 1.27)
-				)
-			)
-		)
-		(property "Description" "Switch, dual pole double throw, separate symbols"
-			(at 190.5 105.41 0)
-			(hide yes)
-			(show_name no)
-			(do_not_autoplace no)
-			(effects
-				(font
-					(size 1.27 1.27)
-				)
-			)
-		)
-		(pin "2"
-		)
-		(pin "4"
-		)
-		(pin "5"
-		)
-		(pin "1"
-		)
-		(pin "3"
-		)
-		(pin "6"
-		)
-		(instances
-			(project "first schematic"
-				(path "/584d0eb4-b791-43e1-a37b-188846e3a37f"
-					(reference "SW1")
-					(unit 2)
-				)
-			)
-		)
 	)
 	(symbol
@@
 	(symbol
 		(lib_id "Switch:SW_DPDT_x2")
-		(at 58.42 107.95 0)
+		(at 58.42 109.22 90)
 		(unit 1)
 		(body_style 1)
@@
 		(fields_autoplaced yes)
 		(property "Reference" "SW1"
-			(at 58.42 99.06 0)
+			(at 63.5 107.9499 90)
 			(show_name no)
 			(do_not_autoplace no)
@@
 					(size 1.27 1.27)
 				)
+				(justify right)
 			)
 		)
 		(property "Value" "SW_DPDT_x2"
-			(at 58.42 101.6 0)
+			(at 63.5 110.4899 90)
 			(show_name no)
 			(do_not_autoplace no)
@@
 					(size 1.27 1.27)
 				)
+				(justify right)
 			)
 		)
 		(property "Footprint" ""
-			(at 58.42 107.95 0)
+			(at 58.42 109.22 0)
 			(hide yes)
 			(show_name no)
@@
 		)
 		(property "Datasheet" ""
-			(at 58.42 107.95 0)
+			(at 58.42 109.22 0)
 			(hide yes)
 			(show_name no)
@@
 		)
 		(property "Description" "Switch, dual pole double throw, separate symbols"
-			(at 58.42 107.95 0)
+			(at 58.42 109.22 0)
 			(hide yes)
 			(show_name no)

Commit message: Autosave
Connections:
- net +3.3V: now also R1.1, R4.1
Other:
- moved on the sheet: BT1
Changed lines of the file:
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@@
 	(generator_version "10.0")
 	(paper "A4")
+	(junction
+		(at 104.14 78.74)
+		(diameter 0)
+		(color 0 0 0 0)
+	)
+	(junction
+		(at 132.08 55.88)
+		(diameter 0)
+		(color 0 0 0 0)
+	)
+	(wire
+		(pts
+			(xy 132.08 55.88) (xy 152.4 55.88)
+		)
+		(stroke
+			(width 0)
+			(type default)
+		)
+	)
+	(wire
+		(pts
+			(xy 152.4 55.88) (xy 152.4 114.3)
+		)
+		(stroke
+			(width 0)
+			(type default)
+		)
+	)
 	(wire
 		(pts
@@
 	(wire
 		(pts
-			(xy 104.14 76.2) (xy 104.14 81.28)
+			(xy 132.08 114.3) (xy 132.08 116.84)
+		)
+		(stroke
+			(width 0)
+			(type default)
+		)
+	)
+	(wire
+		(pts
+			(xy 114.3 78.74) (xy 114.3 55.88)
+		)
+		(stroke
+			(width 0)
+			(type default)
+		)
+	)
+	(wire
+		(pts
+			(xy 104.14 78.74) (xy 104.14 81.28)
+		)
+		(stroke
+			(width 0)
+			(type default)
+		)
+	)
+	(wire
+		(pts
+			(xy 152.4 114.3) (xy 132.08 114.3)
+		)
+		(stroke
+			(width 0)
+			(type default)
+		)
+	)
+	(wire
+		(pts
+			(xy 104.14 78.74) (xy 114.3 78.74)
+		)
+		(stroke
+			(width 0)
+			(type default)
+		)
+	)
+	(wire
+		(pts
+			(xy 104.14 76.2) (xy 104.14 78.74)
+		)
+		(stroke
+			(width 0)
+			(type default)
+		)
+	)
+	(wire
+		(pts
+			(xy 114.3 55.88) (xy 132.08 55.88)
 		)
 		(stroke
@@
 	(symbol
 		(lib_id "Device:Battery_Cell")
-		(at 60.96 88.9 90)
+		(at 57.15 86.36 180)
 		(unit 1)
 		(body_style 1)
@@
 		(fields_autoplaced yes)
 		(property "Reference" "BT1"
-			(at 59.1185 81.28 90)
-			(show_name no)
-			(do_not_autoplace no)
-			(effects
-				(font
-					(size 1.27 1.27)
-				)
+			(at 60.96 86.9314 0)
+			(show_name no)
+			(do_not_autoplace no)
+			(effects
+				(font
+					(size 1.27 1.27)
+				)
+				(justify right)
 			)
 		)
 		(property "Value" "Battery_Cell"
-			(at 59.1185 83.82 90)
-			(show_name no)
-			(do_not_autoplace no)
-			(effects
-				(font
-					(size 1.27 1.27)
-				)
+			(at 60.96 89.4714 0)
+			(show_name no)
+			(do_not_autoplace no)
+			(effects
+				(font
+					(size 1.27 1.27)
+				)
+				(justify right)
 			)
 		)
 		(property "Footprint" ""
-			(at 59.436 88.9 90)
+			(at 57.15 87.884 90)
 			(hide yes)
 			(show_name no)
@@
 		)
 		(property "Datasheet" ""
-			(at 59.436 88.9 90)
+			(at 57.15 87.884 90)
 			(hide yes)
 			(show_name no)
@@
 		)
 		(property "Description" "Single-cell battery"
-			(at 60.96 88.9 0)
+			(at 57.15 86.36 0)
 			(hide yes)
 			(show_name no)
@@
 		)
 		(property "Sim.Device" "V"
-			(at 60.96 88.9 0)
+			(at 57.15 86.36 0)
 			(hide yes)
 			(show_name no)
@@
 		)
 		(property "Sim.Type" "DC"
-			(at 60.96 88.9 0)
+			(at 57.15 86.36 0)
 			(hide yes)
 			(show_name no)
@@
 		)
 		(property "Sim.Pins" "1=+ 2=-"
-			(at 60.96 88.9 0)
-			(hide yes)
-			(show_name no)
+			(at 57.15 86.36 0)
+			(hide yes)
+			(show_name no)

Commit message: Autosave
Connections:
- net +3.3V: now also BT1.1 (+)
- net at SW1.3 (C): now also BT1.2 (-)
Other:
- moved on the sheet: BT1, SW1A
Changed lines of the file:
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@@
+	(wire
+		(pts
+			(xy 104.14 78.74) (xy 57.15 78.74)
+		)
+		(stroke
+			(width 0)
+			(type default)
+		)
+	)
 	(wire
 		(pts
 			(xy 132.08 55.88) (xy 152.4 55.88)
+		)
+		(stroke
+			(width 0)
+			(type default)
+		)
+	)
+	(wire
+		(pts
+			(xy 57.15 78.74) (xy 57.15 83.82)
+		)
+		(stroke
+			(width 0)
+			(type default)
+		)
+	)
+	(wire
+		(pts
+			(xy 57.15 91.44) (xy 57.15 102.87)
 		)
 		(stroke
@@
 	(symbol
 		(lib_id "Switch:SW_DPDT_x2")
-		(at 58.42 109.22 90)
+		(at 54.61 107.95 90)
 		(unit 1)
 		(body_style 1)
@@
 		(fields_autoplaced yes)
 		(property "Reference" "SW1"
-			(at 63.5 107.9499 90)
+			(at 59.69 106.6799 90)
 			(show_name no)
 			(do_not_autoplace no)
@@
 		)
 		(property "Value" "SW_DPDT_x2"
-			(at 63.5 110.4899 90)
+			(at 59.69 109.2199 90)
 			(show_name no)
 			(do_not_autoplace no)
@@
 		)
 		(property "Footprint" ""
-			(at 58.42 109.22 0)
+			(at 54.61 107.95 0)
 			(hide yes)
 			(show_name no)
@@
 		)
 		(property "Datasheet" ""
-			(at 58.42 109.22 0)
+			(at 54.61 107.95 0)
 			(hide yes)
 			(show_name no)
@@
 		)
 		(property "Description" "Switch, dual pole double throw, separate symbols"
-			(at 58.42 109.22 0)
+			(at 54.61 107.95 0)
 			(hide yes)
 			(show_name no)
@@
 	(symbol
 		(lib_id "Device:Battery_Cell")
-		(at 57.15 86.36 180)
+		(at 57.15 88.9 0)
 		(unit 1)
 		(body_style 1)
@@
 		(fields_autoplaced yes)
 		(property "Reference" "BT1"
-			(at 60.96 86.9314 0)
-			(show_name no)
-			(do_not_autoplace no)
-			(effects
-				(font
-					(size 1.27 1.27)
-				)
-				(justify right)
+			(at 60.96 85.7884 0)
+			(show_name no)
+			(do_not_autoplace no)
+			(effects
+				(font
+					(size 1.27 1.27)
+				)
+				(justify left)
 			)
 		)
 		(property "Value" "Battery_Cell"
-			(at 60.96 89.4714 0)
-			(show_name no)
-			(do_not_autoplace no)
-			(effects
-				(font
-					(size 1.27 1.27)
-				)
-				(justify right)
+			(at 60.96 88.3284 0)
+			(show_name no)
+			(do_not_autoplace no)
+			(effects
+				(font
+					(size 1.27 1.27)
+				)
+				(justify left)
 			)
 		)
 		(property "Footprint" ""
-			(at 57.15 87.884 90)
+			(at 57.15 87.376 90)
 			(hide yes)
 			(show_name no)
@@
 		)
 		(property "Datasheet" ""
-			(at 57.15 87.884 90)
+			(at 57.15 87.376 90)
 			(hide yes)
 			(show_name no)
@@
 		)
 		(property "Description" "Single-cell battery"
-			(at 57.15 86.36 0)
+			(at 57.15 88.9 0)
 			(hide yes)
 			(show_name no)
@@
 		)
 		(property "Sim.Device" "V"
-			(at 57.15 86.36 0)
+			(at 57.15 88.9 0)
 			(hide yes)
 			(show_name no)
@@
 		)
 		(property "Sim.Type" "DC"
-			(at 57.15 86.36 0)
+			(at 57.15 88.9 0)
 			(hide yes)
 			(show_name no)
@@
 		)
 		(property "Sim.Pins" "1=+ 2=-"
-			(at 57.15 86.36 0)
-			(hide yes)
-			(show_name no)
+			(at 57.15 88.9 0)
+			(hide yes)
+			(show_name no)

Commit message: Autosave
Connections:
- net at R1.2: now also R3.1, U1.3 (XTAL2/PB4)
- net at R3.2: now also MK1.1 (-)
Changed lines of the file:
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@@
 		(color 0 0 0 0)
+	)
+	(junction
+		(at 132.08 63.5)
+		(diameter 0)
+		(color 0 0 0 0)
+	)
+	(wire
+		(pts
+			(xy 132.08 80.01) (xy 165.1 80.01)
+		)
+		(stroke
+			(width 0)
+			(type default)
+		)
 	)
 	(wire
@@
 	(wire
 		(pts
+			(xy 165.1 142.24) (xy 132.08 142.24)
+		)
+		(stroke
+			(width 0)
+			(type default)
+		)
+	)
+	(wire
+		(pts
 			(xy 152.4 55.88) (xy 152.4 114.3)
 		)
@@
 	(wire
 		(pts
+			(xy 165.1 80.01) (xy 165.1 142.24)
+		)
+		(stroke
+			(width 0)
+			(type default)
+		)
+	)
+	(wire
+		(pts
 			(xy 132.08 114.3) (xy 132.08 116.84)
 		)
@@
 	(wire
 		(pts
+			(xy 132.08 63.5) (xy 132.08 72.39)
+		)
+		(stroke
+			(width 0)
+			(type default)
+		)
+	)
+	(wire
+		(pts
 			(xy 114.3 78.74) (xy 114.3 55.88)
+		)
+		(stroke
+			(width 0)
+			(type default)
+		)
+	)
+	(wire
+		(pts
+			(xy 119.38 99.06) (xy 127 99.06)
 		)
 		(stroke
@@
 	(wire
 		(pts
+			(xy 127 99.06) (xy 127 63.5)
+		)
+		(stroke
+			(width 0)
+			(type default)
+		)
+	)
+	(wire
+		(pts
 			(xy 104.14 76.2) (xy 104.14 78.74)
 		)
 		(stroke
+			(width 0)
+			(type default)
+		)
+	)
+	(wire
+		(pts
+			(xy 127 63.5) (xy 132.08 63.5)
+		)
+		(stroke

Commit message: Autosave
Connections:
- net GND: now also MK1.1 (-), R3.2, SW1.2 (B)
Changed lines of the file:
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@@
 	(paper "A4")
 	(junction
+		(at 104.14 115.57)
+		(diameter 0)
+		(color 0 0 0 0)
+	)
+	(junction
+		(at 132.08 142.24)
+		(diameter 0)
+		(color 0 0 0 0)
+	)
+	(junction
 		(at 104.14 78.74)
 		(diameter 0)
@@
 	(wire
 		(pts
-			(xy 104.14 111.76) (xy 104.14 118.11)
+			(xy 54.61 113.03) (xy 54.61 115.57)
+		)
+		(stroke
+			(width 0)
+			(type default)
+		)
+	)
+	(wire
+		(pts
+			(xy 104.14 111.76) (xy 104.14 115.57)
+		)
+		(stroke
+			(width 0)
+			(type default)
+		)
+	)
+	(wire
+		(pts
+			(xy 114.3 115.57) (xy 104.14 115.57)
+		)
+		(stroke
+			(width 0)
+			(type default)
+		)
+	)
+	(wire
+		(pts
+			(xy 132.08 142.24) (xy 114.3 142.24)
 		)
 		(stroke
@@
 	(wire
 		(pts
+			(xy 104.14 115.57) (xy 54.61 115.57)
+		)
+		(stroke
+			(width 0)
+			(type default)
+		)
+	)
+	(wire
+		(pts
 			(xy 104.14 78.74) (xy 104.14 81.28)
 		)
@@
 	(wire
 		(pts
+			(xy 114.3 142.24) (xy 114.3 115.57)
+		)
+		(stroke
+			(width 0)
+			(type default)
+		)
+	)
+	(wire
+		(pts
 			(xy 127 99.06) (xy 127 63.5)
 		)
 		(stroke
+			(width 0)
+			(type default)
+		)
+	)
+	(wire
+		(pts
+			(xy 104.14 115.57) (xy 104.14 118.11)
+		)
+		(stroke

Commit message: SCH Save
Connections:
- net GND: now also R2.2
- net at U1.6 (PB1): now also D1.2 (A)
- net at U1.7 (PB2): now also MK1.2 (+), R4.2
- net at R2.1: now also D1.1 (K)
Changed lines of the file:
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@@
+	)
+	(junction
+		(at 132.08 124.46)
+		(diameter 0)
+		(color 0 0 0 0)
 	)
 	(junction
@@
 	)
 	(junction
+		(at 165.1 109.22)
+		(diameter 0)
+		(color 0 0 0 0)
+	)
+	(junction
 		(at 132.08 55.88)
 		(diameter 0)
@@
 	(wire
 		(pts
+			(xy 132.08 109.22) (xy 165.1 109.22)
+		)
+		(stroke
+			(width 0)
+			(type default)
+		)
+	)
+	(wire
+		(pts
 			(xy 104.14 78.74) (xy 57.15 78.74)
 		)
@@
 	(wire
 		(pts
+			(xy 165.1 109.22) (xy 165.1 142.24)
+		)
+		(stroke
+			(width 0)
+			(type default)
+		)
+	)
+	(wire
+		(pts
 			(xy 132.08 55.88) (xy 152.4 55.88)
 		)
@@
 	(wire
 		(pts
+			(xy 132.08 86.36) (xy 125.73 86.36)
+		)
+		(stroke
+			(width 0)
+			(type default)
+		)
+	)
+	(wire
+		(pts
 			(xy 114.3 115.57) (xy 104.14 115.57)
 		)
@@
 	(wire
 		(pts
+			(xy 132.08 93.98) (xy 132.08 101.6)
+		)
+		(stroke
+			(width 0)
+			(type default)
+		)
+	)
+	(wire
+		(pts
+			(xy 128.27 93.98) (xy 128.27 124.46)
+		)
+		(stroke
+			(width 0)
+			(type default)
+		)
+	)
+	(wire
+		(pts
 			(xy 132.08 142.24) (xy 114.3 142.24)
 		)
@@
 	(wire
 		(pts
-			(xy 165.1 80.01) (xy 165.1 142.24)
+			(xy 165.1 80.01) (xy 165.1 109.22)
 		)
 		(stroke
@@
 	(wire
 		(pts
+			(xy 128.27 124.46) (xy 132.08 124.46)
+		)
+		(stroke
+			(width 0)
+			(type default)
+		)
+	)
+	(wire
+		(pts
+			(xy 132.08 124.46) (xy 132.08 132.08)
+		)
+		(stroke
+			(width 0)
+			(type default)
+		)
+	)
+	(wire
+		(pts
 			(xy 119.38 99.06) (xy 127 99.06)
 		)
@@
 	(wire
 		(pts
+			(xy 119.38 91.44) (xy 125.73 91.44)
+		)
+		(stroke
+			(width 0)
+			(type default)
+		)
+	)
+	(wire
+		(pts
 			(xy 104.14 115.57) (xy 54.61 115.57)
 		)
@@
 	(wire
 		(pts
+			(xy 119.38 93.98) (xy 128.27 93.98)
+		)
+		(stroke
+			(width 0)
+			(type default)
+		)
+	)
+	(wire
+		(pts
 			(xy 104.14 78.74) (xy 114.3 78.74)
 		)
 		(stroke
+			(width 0)
+			(type default)
+		)
+	)
+	(wire
+		(pts
+			(xy 125.73 86.36) (xy 125.73 91.44)
+		)
+		(stroke

Commit message: SCH Save
Parts:
- BT1: value Battery_Cell -> 3.3V Cell
- D1: value LED -> 5mm Yellow LED
- R1: value R -> 10k
- R2: renamed from R3; value LDR07 -> 5mm LDR
- R3: renamed from R4; value R -> 5.6k
- R4: renamed from R2; value R -> 470R
- SW1: value SW_DPDT_x2 -> Slide Switch
Connections:
- net +3.3V: now also D1.2 (A)
- net LDR: now reaches R1.2, R2.1
- net LDR: now also U1.2 (XTAL1/PB3); no longer U1.3 (XTAL2/PB4)
- net at U1.6 (PB1): no longer D1.2 (A)
- net MIC: now reaches MK1.2 (+), R3.2
- net MIC: now also U1.3 (XTAL2/PB4); no longer U1.7 (PB2)
- net at R4.1: no longer D1.1 (K)
- net at SW1.3 (C): no longer BT1.2 (-)
- new net LED: U1.7 (PB2)
- no-connect marks 0 -> 3
Other:
- note added: "Battery Unit"
- note added: "Light Sensing Unit"
- note added: "Light Unit"
- note added: "Microcontroller Unit"
- note added: "Sound Sensing Unit"
- company: (none) -> PCB Cupid
- title: (none) -> Digital Diya
- moved on the sheet: BT1, D1, MK1, R1, R2, R3, R4, SW1A, U1
